Commit message: new

File: ur.urdf.xacro (robot description, xacro)
@@ -41,5 +41,5 @@
     <visual>
       <geometry>
-        <box size="0.05 0.05 0.05"/>
+        <box size="0.03 0.03 0.03"/>
       </geometry>
     </visual>
@@ -48,5 +48,5 @@
     <parent link="tool0"/>
     <child link="camera_link"/>
-    <origin xyz="0 0 0.10" rpy="0 0 0"/>
+    <origin xyz="0.0 0.10 0.10" rpy="0 0 0"/>
   </joint>
   <!-- ================================================ -->
